File: electronics/mainboard/mainboard.kicad_pcb (KiCad board)
At the start: 2 copper layers, 151.8 x 54.6 mm, 52 parts, among them J1 Conn_01x09, J10 Conn_01x08, J11 Conn_01x08, J12 Conn_01x08, J13 Conn_02x18_Odd_Even, J14 Conn_01x08, J15 Conn_01x08, J16 Conn_01x10, J17 Conn_02x03_Odd_Even, J2 Conn_01x09, J3 Conn_01x09, J4 Conn_01x09, J5 Conn_01x09, J6 Conn_01x09, J7 Conn_01x09, J8 Conn_01x09, J9 Conn_01x09

Commit message: drc check pass
Parts:
- added REF**: MountingHole_3.2mm_M3, MountingHole:MountingHole_3.2mm_M3, F.Cu at (52.1, 112.4)
- added REF**: MountingHole_3.2mm_M3, MountingHole:MountingHole_3.2mm_M3, F.Cu at (52.1, 66.7)
- moved NT5 3.72 mm to (170.8, 71.1)
- moved NT8 3.08 mm to (122.6, 70.5)
- moved NT9 3.08 mm to (109.9, 70.5)
- moved NT6 2.44 mm to (168.3, 69.8)
- moved NT7 2.44 mm to (141.0, 88.3)
- moved NT1 2.32 mm to (175.4, 68.6), turned to 180 degrees
- moved NT2 1.81 mm to (141.6, 93.3)
- moved NT4 1.18 mm to (185.0, 110.5)
- moved NT3 1.17 mm to (111.8, 113.7)
Connections:
- XA1 pad : (no net) -> unconnected-(J10-Pad1)
Routing:
- net GND: track 7.14 -> 22.1 mm
- net /5V1: track 0.00 -> 3.17 mm
- net /GND3: track 0.00 -> 2.44 mm
- net /GND4: track 0.00 -> 2.32 mm
- net /5V2: track 0.00 -> 1.68 mm
- net /5V4: track 0.00 -> 1.17 mm
