File: electronics/mainboard/mainboard.kicad_pcb (KiCad board)
At the start: 2 copper layers, 151.8 x 54.6 mm, 54 parts, among them J1 Conn_01x09, J10 Conn_01x08, J11 Conn_01x08, J12 Conn_01x08, J13 Conn_02x18_Odd_Even, J14 Conn_01x08, J15 Conn_01x08, J16 Conn_01x10, J17 Conn_02x03_Odd_Even, J2 Conn_01x09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

Commit message: add project and version information
Other:
- board text added: "${PROJECT} ${PROJECT-URL} tag: ${GIT-COMMIT-TAG} | commit: ${GIT-COMMIT-HASH}"
Changed lines of the file:
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@@
   )
   (paper "A4")
+  (title_block
+    (title "Mainboard")
+    (comment 1 "${PROJECT}")
+    (comment 2 "${PROJECT-URL}")
+    (comment 3 "${GIT-COMMIT-HASH}")
+    (comment 4 "${GIT-COMMIT-TAG}")
+  )
   (layers
     (0 "F.Cu" signal)
@@
     )
   )
+  (property "GIT-COMMIT-HASH" "noHash")
+  (property "GIT-COMMIT-TAG" "noTag")
+  (property "PROJECT" "Light Installation - Mainboard")
+  (property "PROJECT-URL" "https://github.com/erichstuder/Light_Installation")
   (net 0 "")
   (net 1 "+5V")
@@
   (gr_line (start 199.39 116.84) (end 47.625 116.84) (layer "Edge.Cuts") (width 0.1))
   (gr_line (start 199.39 62.23) (end 199.39 116.84) (layer "Edge.Cuts") (width 0.1))
+  (gr_text "${PROJECT}\n${PROJECT-URL}\ntag: ${GIT-COMMIT-TAG} | commit: ${GIT-COMMIT-HASH}" (at 57.15 66.04) (layer "F.SilkS")
+    (effects (font (size 1.2 1.2) (thickness 0.15)) (justify left))
+  )
   (segment (start 56.515 81.28) (end 57.5075 81.28) (width 0.25) (layer "B.Cu") (net 2))
   (segment (start 56.18 80.945) (end 56.515 81.28) (width 0.25) (layer "B.Cu") (net 2))

Commit message: solve erc and drc problems
Parts:
- removed REF** (x2): MountingHole_3.2mm_M3, MountingHole:MountingHole_3.2mm_M3
- added H1: MountingHole, MountingHole:MountingHole_3.2mm_M3, F.Cu at (52.1, 66.7)
- added H2: MountingHole, MountingHole:MountingHole_3.2mm_M3, F.Cu at (52.1, 112.4)
